Commit message: Untested Model

File: src/ahser_description/urdf/ahser.urdf.xacro (robot description, xacro)
@@ -1,10 +1,187 @@
 <?xml version="1.0"?>
 <robot xmlns:xacro="http://www.ros.org/wiki/xacro" name="ahser">
-  <!-- AHSER: Autonomous Hospital Service Robot -->
-  <!-- Top-level robot description file -->
-  <xacro:include filename="$(find ahser_description)/urdf/materials.xacro" />
-  <xacro:include filename="$(find ahser_description)/urdf/wheels.xacro" />
-  <xacro:include filename="$(find ahser_description)/urdf/sensors.xacro" />
-  <!-- Base link frame definition (physical/visual geometry to be added in modeling phase) -->
-  <link name="base_link" />
+  <!-- ==================================================================== -->
+  <!-- AHSER: Autonomous Hospital Service Robot                             -->
+  <!-- Top-Level System URDF / XACRO Description                            -->
+  <!-- ==================================================================== -->
+  <!-- ==================================================================== -->
+  <!-- Centralized Robot Dimensional & Mass Parameters (SI Metric Units)    -->
+  <!-- ==================================================================== -->
+  <!-- Ground clearance and wheel parameters -->
+  <xacro:property name="wheel_radius" value="0.080"/>       <!-- 80 mm radius / 160 mm diameter -->
+  <xacro:property name="wheel_width" value="0.040"/>        <!-- 40 mm tread width -->
+  <xacro:property name="wheel_track" value="0.380"/>        <!-- 380 mm lateral track width between wheels -->
+  <xacro:property name="wheel_mass" value="0.80"/>          <!-- 0.80 kg per drive wheel -->
+  <xacro:property name="ground_clearance" value="0.030"/>   <!-- 30 mm chassis underside ground clearance -->
+  <xacro:property name="caster_radius" value="0.030"/>      <!-- 30 mm radius caster sphere (touches z=0) -->
+  <xacro:property name="caster_x_offset" value="0.180"/>    <!-- 180 mm fore/aft distance from axle -->
+  <xacro:property name="caster_mass" value="0.25"/>         <!-- 0.25 kg per caster assembly -->
+  <!-- Main chassis body parameters -->
+  <xacro:property name="chassis_length" value="0.480"/>     <!-- 480 mm front-to-back length -->
+  <xacro:property name="chassis_width" value="0.320"/>      <!-- 320 mm width (fits between wheels) -->
+  <xacro:property name="chassis_height" value="0.180"/>     <!-- 180 mm vertical height -->
+  <xacro:property name="chassis_mass" value="8.00"/>        <!-- 8.0 kg base chassis structure and battery -->
+  <!-- Upper medicine/storage compartment parameters -->
+  <xacro:property name="storage_length" value="0.340"/>     <!-- 340 mm storage cabinet length -->
+  <xacro:property name="storage_width" value="0.280"/>      <!-- 280 mm storage cabinet width -->
+  <xacro:property name="storage_height" value="0.260"/>     <!-- 260 mm storage cabinet height -->
+  <xacro:property name="storage_x_offset" value="-0.020"/>  <!-- Offset slightly aft for front sensor deck -->
+  <xacro:property name="storage_mass" value="3.50"/>        <!-- 3.5 kg payload compartment -->
+  <!-- Sensor parameters -->
+  <xacro:property name="lidar_radius" value="0.038"/>       <!-- 76 mm diameter LiDAR housing -->
+  <xacro:property name="lidar_height" value="0.040"/>       <!-- 40 mm LiDAR sensor height -->
+  <xacro:property name="lidar_mass" value="0.25"/>          <!-- 0.25 kg 2D LiDAR scanner -->
+  <xacro:property name="lidar_x_offset" value="0.060"/>     <!-- Forward-biased on roof for clear front view -->
+  <xacro:property name="lidar_z_offset"
+    value="${ground_clearance + chassis_height + storage_height + lidar_height / 2.0}"/>
+  <xacro:property name="camera_length" value="0.030"/>
+  <xacro:property name="camera_width" value="0.080"/>
+  <xacro:property name="camera_height" value="0.030"/>
+  <xacro:property name="camera_mass" value="0.10"/>
+  <xacro:property name="camera_x_offset" value="${chassis_length / 2.0 + camera_length / 2.0}"/>
+  <xacro:property name="camera_z_offset" value="${ground_clearance + chassis_height * 0.82}"/>
+  <xacro:property name="imu_size" value="0.025"/>
+  <xacro:property name="imu_height" value="0.008"/>
+  <xacro:property name="imu_mass" value="0.02"/>
+  <xacro:property name="imu_x_offset" value="0.000"/>
+  <xacro:property name="imu_z_offset" value="${ground_clearance + 0.020}"/>
+  <!-- ==================================================================== -->
+  <!-- Modular Includes                                                     -->
+  <!-- ==================================================================== -->
+  <xacro:include filename="$(find ahser_description)/urdf/materials.xacro"/>
+  <xacro:include filename="$(find ahser_description)/urdf/wheels.xacro"/>
+  <xacro:include filename="$(find ahser_description)/urdf/sensors.xacro"/>
+  <!-- ==================================================================== -->
+  <!-- Kinematic Base / Footprint Frames                                    -->
+  <!-- ==================================================================== -->
+  <!-- Root Link: base_link located at ground plane projection of drive axle -->
+  <link name="base_link"/>
+  <!-- base_footprint on ground plane z=0 (REP 120 standard) -->
+  <joint name="base_footprint_joint" type="fixed">
+    <parent link="base_link"/>
+    <child link="base_footprint"/>
+    <origin xyz="0 0 0" rpy="0 0 0"/>
+  </joint>
+  <link name="base_footprint"/>
+  <!-- ==================================================================== -->
+  <!-- Main Chassis Link & Joint                                            -->
+  <!-- ==================================================================== -->
+  <joint name="chassis_joint" type="fixed">
+    <parent link="base_link"/>
+    <child link="chassis_link"/>
+    <!-- Positioned above ground clearance -->
+    <origin xyz="0.0 0.0 ${ground_clearance + chassis_height / 2.0}" rpy="0 0 0"/>
+  </joint>
+  <link name="chassis_link">
+    <!-- Main white chassis body enclosure -->
+    <visual>
+      <origin xyz="0 0 0" rpy="0 0 0"/>
+      <geometry>
+        <box size="${chassis_length} ${chassis_width} ${chassis_height}"/>
+      </geometry>
+      <material name="hospital_white"/>
+    </visual>
+    <!-- Lower protective perimeter bumper / skirt -->
+    <visual>
+      <origin xyz="0 0 -${chassis_height * 0.35}" rpy="0 0 0"/>
+      <geometry>
+        <box size="${chassis_length + 0.015} ${chassis_width + 0.015} ${chassis_height * 0.30}"/>
+      </geometry>
+      <material name="dark_grey"/>
+    </visual>
+    <!-- Medical teal accent beltline trim -->
+    <visual>
+      <origin xyz="0 0 ${chassis_height * 0.35}" rpy="0 0 0"/>
+      <geometry>
+        <box size="${chassis_length + 0.006} ${chassis_width + 0.006} 0.015"/>
+      </geometry>
+      <material name="medical_teal"/>
+    </visual>
+    <!-- Physical collision bounding box -->
+    <collision>
+      <origin xyz="0 0 0" rpy="0 0 0"/>
+      <geometry>
+        <box size="${chassis_length} ${chassis_width} ${chassis_height}"/>
+      </geometry>
+    </collision>
+    <!-- Chassis inertial tensor -->
+    <inertial>
+      <mass value="${chassis_mass}"/>
+      <origin xyz="0 0 0" rpy="0 0 0"/>
+      <inertia
+        ixx="${(chassis_mass / 12.0) * (chassis_width * chassis_width + chassis_height * chassis_height)}"
+        ixy="0.0"
+        ixz="0.0"
+        iyy="${(chassis_mass / 12.0) * (chassis_length * chassis_length + chassis_height * chassis_height)}"
+        iyz="0.0"
+        izz="${(chassis_mass / 12.0) * (chassis_length * chassis_length + chassis_width * chassis_width)}"/>
+    </inertial>
+  </link>
+  <!-- ==================================================================== -->
+  <!-- Upper Medicine / Supply Storage Compartment                          -->
+  <!-- ==================================================================== -->
+  <joint name="storage_compartment_joint" type="fixed">
+    <parent link="base_link"/>
+    <child link="storage_compartment_link"/>
+    <!-- Stacked directly upon the chassis top surface -->
+    <origin xyz="${storage_x_offset} 0.0 ${ground_clearance + chassis_height + storage_height / 2.0}" rpy="0 0 0"/>
+  </joint>
+  <link name="storage_compartment_link">
+    <!-- Storage cabinet exterior body -->
+    <visual>
+      <origin xyz="0 0 0" rpy="0 0 0"/>
+      <geometry>
+        <box size="${storage_length} ${storage_width} ${storage_height}"/>
+      </geometry>
+      <material name="hospital_white"/>
+    </visual>
+    <!-- Front medicine delivery door face with medical teal styling -->
+    <visual>
+      <origin xyz="${storage_length / 2.0 + 0.002} 0 0" rpy="0 0 0"/>
+      <geometry>
+        <box size="0.004 ${storage_width * 0.85} ${storage_height * 0.80}"/>
+      </geometry>
+      <material name="medical_teal"/>
+    </visual>
+    <!-- Storage door latch / handle visual indicator -->
+    <visual>
+      <origin xyz="${storage_length / 2.0 + 0.006} ${storage_width * 0.3} 0" rpy="0 0 0"/>
+      <geometry>
+        <box size="0.008 0.015 0.080"/>
+      </geometry>
+      <material name="dark_grey"/>
+    </visual>
+    <!-- Physical collision bounding box -->
+    <collision>
+      <origin xyz="0 0 0" rpy="0 0 0"/>
+      <geometry>
+        <box size="${storage_length} ${storage_width} ${storage_height}"/>
+      </geometry>
+    </collision>
+    <!-- Storage compartment inertial tensor -->
+    <inertial>
+      <mass value="${storage_mass}"/>
+      <origin xyz="0 0 0" rpy="0 0 0"/>
+      <inertia
+        ixx="${(storage_mass / 12.0) * (storage_width * storage_width + storage_height * storage_height)}"
+        ixy="0.0"
+        ixz="0.0"
+        iyy="${(storage_mass / 12.0) * (storage_length * storage_length + storage_height * storage_height)}"
+        iyz="0.0"
+        izz="${(storage_mass / 12.0) * (storage_length * storage_length + storage_width * storage_width)}"/>
+    </inertial>
+  </link>
+  <!-- ==================================================================== -->
+  <!-- Wheels: Powered Drive Wheels & Passive Stability Casters             -->
+  <!-- ==================================================================== -->
+  <!-- Left & Right Differential Drive Wheels -->
+  <xacro:drive_wheel prefix="left" y_reflect="1"/>
+  <xacro:drive_wheel prefix="right" y_reflect="-1"/>
+  <!-- Front & Rear Passive Support Casters for balanced 4-point ground contact -->
+  <xacro:caster_wheel prefix="front" x_offset="${caster_x_offset}"/>
+  <xacro:caster_wheel prefix="rear" x_offset="-${caster_x_offset}"/>
+  <!-- ==================================================================== -->
+  <!-- Sensor Suite (LiDAR, RGB Camera, IMU)                                -->
+  <!-- ==================================================================== -->
+  <xacro:sensors/>
 </robot>

File: src/ahser_description/urdf/materials.xacro (robot description, xacro)
@@ -1,16 +1,39 @@
 <?xml version="1.0"?>
 <robot xmlns:xacro="http://www.ros.org/wiki/xacro">
-  <!-- AHSER Material Color Definitions -->
-  <material name="white">
-    <color rgba="1.0 1.0 1.0 1.0"/>
+  <!-- ==================================================================== -->
+  <!-- AHSER Material & Color Definitions                                  -->
+  <!-- Clean, professional medical/service robot color palette             -->
+  <!-- ==================================================================== -->
+  <!-- Primary Chassis & Storage Body: Clean Hospital White -->
+  <material name="hospital_white">
+    <color rgba="0.92 0.94 0.96 1.0"/>
   </material>
+  <!-- Accent: Medical Service Teal/Cyan for Doors & Brand Identification -->
+  <material name="medical_teal">
+    <color rgba="0.0 0.60 0.65 1.0"/>
+  </material>
+  <!-- Chassis Lower Skirt & Mechanical Mounts: Dark Graphite Grey -->
   <material name="dark_grey">
-    <color rgba="0.2 0.2 0.2 1.0"/>
+    <color rgba="0.22 0.22 0.25 1.0"/>
   </material>
-  <material name="hospital_blue">
-    <color rgba="0.0 0.45 0.73 1.0"/>
+  <!-- Secondary Trims & Structural Plates: Neutral Light Grey -->
+  <material name="light_grey">
+    <color rgba="0.75 0.77 0.80 1.0"/>
   </material>
-  <material name="black">
-    <color rgba="0.05 0.05 0.05 1.0"/>
+  <!-- Drive Wheel Tires: Durable Matte Rubber Black -->
+  <material name="wheel_black">
+    <color rgba="0.12 0.12 0.12 1.0"/>
+  </material>
+  <!-- Passive Caster Spheres: Smooth Low-Friction Metallic Steel -->
+  <material name="caster_metallic">
+    <color rgba="0.65 0.65 0.68 1.0"/>
+  </material>
+  <!-- Sensor Enclosures (LiDAR, Camera body): Matte Black -->
+  <material name="sensor_black">
+    <color rgba="0.10 0.10 0.10 1.0"/>
+  </material>
+  <!-- Optical Lenses & Display Panel: Tinted Obsidian -->
+  <material name="lens_glass">
+    <color rgba="0.05 0.05 0.08 1.0"/>
   </material>
 </robot>

File: src/ahser_description/urdf/sensors.xacro (robot description, xacro)
@@ -1,5 +1,133 @@
 <?xml version="1.0"?>
 <robot xmlns:xacro="http://www.ros.org/wiki/xacro">
-  <!-- AHSER Sensor Definitions -->
-  <!-- LiDAR, Depth Camera, and IMU macros will be implemented in the robot modeling phase -->
+  <!-- ==================================================================== -->
+  <!-- AHSER Perception & Localization Sensor Suite                        -->
+  <!-- Frames and primitive visual/collision models for LiDAR, Camera, IMU  -->
+  <!-- ==================================================================== -->
+  <xacro:macro name="sensors">
+    <!-- Top-Mounted 2D Planar LiDAR -->
+    <joint name="lidar_joint" type="fixed">
+      <parent link="base_link"/>
+      <child link="lidar_link"/>
+      <!-- Elevated on the roof of the upper storage compartment for 360-deg FOV -->
+      <origin xyz="${lidar_x_offset} 0.0 ${lidar_z_offset}" rpy="0 0 0"/>
+    </joint>
+    <link name="lidar_link">
+      <!-- LiDAR Base Collar -->
+      <visual>
+        <origin xyz="0 0 0" rpy="0 0 0"/>
+        <geometry>
+          <cylinder radius="${lidar_radius}" length="${lidar_height}"/>
+        </geometry>
+        <material name="sensor_black"/>
+      </visual>
+      <!-- LiDAR Rotating Optical Head Accent -->
+      <visual>
+        <origin xyz="0 0 ${lidar_height * 0.25}" rpy="0 0 0"/>
+        <geometry>
+          <cylinder radius="${lidar_radius * 0.9}" length="${lidar_height * 0.4}"/>
+        </geometry>
+        <material name="medical_teal"/>
+      </visual>
+      <collision>
+        <origin xyz="0 0 0" rpy="0 0 0"/>
+        <geometry>
+          <cylinder radius="${lidar_radius}" length="${lidar_height}"/>
+        </geometry>
+      </collision>
+      <inertial>
+        <mass value="${lidar_mass}"/>
+        <origin xyz="0 0 0" rpy="0 0 0"/>
+        <inertia
+          ixx="${(lidar_mass / 12.0) * (3.0 * lidar_radius * lidar_radius + lidar_height * lidar_height)}"
+          ixy="0.0"
+          ixz="0.0"
+          iyy="${(lidar_mass / 12.0) * (3.0 * lidar_radius * lidar_radius + lidar_height * lidar_height)}"
+          iyz="0.0"
+          izz="${(lidar_mass / 2.0) * (lidar_radius * lidar_radius)}"/>
+      </inertial>
+    </link>
+    <!-- Front-Facing RGB Perception Camera -->
+    <joint name="camera_joint" type="fixed">
+      <parent link="base_link"/>
+      <child link="camera_link"/>
+      <!-- Mounted on the upper-front brow of the chassis facing forward (+X) -->
+      <origin xyz="${camera_x_offset} 0.0 ${camera_z_offset}" rpy="0 0 0"/>
+    </joint>
+    <link name="camera_link">
+      <!-- Camera Body Enclosure -->
+      <visual>
+        <origin xyz="0 0 0" rpy="0 0 0"/>
+        <geometry>
+          <box size="${camera_length} ${camera_width} ${camera_height}"/>
+        </geometry>
+        <material name="sensor_black"/>
+      </visual>
+      <!-- Camera Lens Barrel -->
+      <visual>
+        <origin xyz="${camera_length / 2.0 + 0.003} 0 0" rpy="0 ${pi/2} 0"/>
+        <geometry>
+          <cylinder radius="${camera_height * 0.3}" length="0.006"/>
+        </geometry>
+        <material name="lens_glass"/>
+      </visual>
+      <collision>
+        <origin xyz="0 0 0" rpy="0 0 0"/>
+        <geometry>
+          <box size="${camera_length} ${camera_width} ${camera_height}"/>
+        </geometry>
+      </collision>
+      <inertial>
+        <mass value="${camera_mass}"/>
+        <origin xyz="0 0 0" rpy="0 0 0"/>
+        <inertia
+          ixx="${(camera_mass / 12.0) * (camera_width * camera_width + camera_height * camera_height)}"
+          ixy="0.0"
+          ixz="0.0"
+          iyy="${(camera_mass / 12.0) * (camera_length * camera_length + camera_height * camera_height)}"
+          iyz="0.0"
+          izz="${(camera_mass / 12.0) * (camera_length * camera_length + camera_width * camera_width)}"/>
+      </inertial>
+    </link>
+    <!-- Standard ROS Camera Optical Frame (Z forward, X right, Y down) -->
+    <joint name="camera_optical_joint" type="fixed">
+      <parent link="camera_link"/>
+      <child link="camera_optical_link"/>
+      <origin xyz="0 0 0" rpy="-${pi/2} 0 -${pi/2}"/>
+    </joint>
+    <link name="camera_optical_link"/>
+    <!-- Inertial Measurement Unit (IMU) -->
+    <joint name="imu_joint" type="fixed">
+      <parent link="base_link"/>
+      <child link="imu_link"/>
+      <!-- Positioned close to the geometric center and drive axle -->
+      <origin xyz="${imu_x_offset} 0.0 ${imu_z_offset}" rpy="0 0 0"/>
+    </joint>
+    <link name="imu_link">
+      <visual>
+        <origin xyz="0 0 0" rpy="0 0 0"/>
+        <geometry>
+          <box size="${imu_size} ${imu_size} ${imu_height}"/>
+        </geometry>
+        <material name="dark_grey"/>
+      </visual>
+      <collision>
+        <origin xyz="0 0 0" rpy="0 0 0"/>
+        <geometry>
+          <box size="${imu_size} ${imu_size} ${imu_height}"/>
+        </geometry>
+      </collision>
+      <inertial>
+        <mass value="${imu_mass}"/>
+        <origin xyz="0 0 0" rpy="0 0 0"/>
+        <inertia
+          ixx="${(imu_mass / 12.0) * (imu_size * imu_size + imu_height * imu_height)}"
+          ixy="0.0"
+          ixz="0.0"
+          iyy="${(imu_mass / 12.0) * (imu_size * imu_size + imu_height * imu_height)}"
+          iyz="0.0"
+          izz="${(imu_mass / 12.0) * (imu_size * imu_size + imu_size * imu_size)}"/>
+      </inertial>
+    </link>
+  </xacro:macro>
 </robot>

File: src/ahser_description/urdf/wheels.xacro (robot description, xacro)
@@ -1,5 +1,92 @@
 <?xml version="1.0"?>
 <robot xmlns:xacro="http://www.ros.org/wiki/xacro">
-  <!-- AHSER Wheel Definitions -->
-  <!-- Drive wheel and caster wheel macros will be implemented in the robot modeling phase -->
+  <!-- ==================================================================== -->
+  <!-- AHSER Wheels & Mobile Base Locomotion Module                        -->
+  <!-- Differential drive powered wheels and passive caster support wheels  -->
+  <!-- ==================================================================== -->
+  <!-- Macro: Differential Drive Powered Wheel -->
+  <xacro:macro name="drive_wheel" params="prefix y_reflect">
+    <joint name="${prefix}_wheel_joint" type="continuous">
+      <parent link="base_link"/>
+      <child link="${prefix}_wheel_link"/>
+      <!-- Symmetrical placement along the transverse (Y) axle -->
+      <origin xyz="0.0 ${y_reflect * (wheel_track / 2.0)} ${wheel_radius}" rpy="0 0 0"/>
+      <!-- Standard ROS differential drive rotation axis (Pitch / Y-axis) -->
+      <axis xyz="0 1 0"/>
+      <dynamics damping="0.1" friction="0.1"/>
+    </joint>
+    <link name="${prefix}_wheel_link">
+      <visual>
+        <!-- Rotate cylinder from Z to Y axis -->
+        <origin xyz="0 0 0" rpy="${pi/2} 0 0"/>
+        <geometry>
+          <cylinder radius="${wheel_radius}" length="${wheel_width}"/>
+        </geometry>
+        <material name="wheel_black"/>
+      </visual>
+      <collision>
+        <origin xyz="0 0 0" rpy="${pi/2} 0 0"/>
+        <geometry>
+          <cylinder radius="${wheel_radius}" length="${wheel_width}"/>
+        </geometry>
+      </collision>
+      <!-- Accurate cylinder inertia aligned with rotation axis Y -->
+      <inertial>
+        <mass value="${wheel_mass}"/>
+        <origin xyz="0 0 0" rpy="0 0 0"/>
+        <inertia
+          ixx="${(wheel_mass / 12.0) * (3.0 * wheel_radius * wheel_radius + wheel_width * wheel_width)}"
+          ixy="0.0"
+          ixz="0.0"
+          iyy="${(wheel_mass / 2.0) * (wheel_radius * wheel_radius)}"
+          iyz="0.0"
+          izz="${(wheel_mass / 12.0) * (3.0 * wheel_radius * wheel_radius + wheel_width * wheel_width)}"/>
+      </inertial>
+    </link>
+  </xacro:macro>
+  <!-- Macro: Passive Support Caster Wheel -->
+  <xacro:macro name="caster_wheel" params="prefix x_offset">
+    <joint name="${prefix}_caster_joint" type="fixed">
+      <parent link="base_link"/>
+      <child link="${prefix}_caster_link"/>
+      <!-- Positioned along sagittal centerline (X) at height caster_radius to touch ground -->
+      <origin xyz="${x_offset} 0.0 ${caster_radius}" rpy="0 0 0"/>
+    </joint>
+    <link name="${prefix}_caster_link">
+      <!-- Caster rolling sphere -->
+      <visual>
+        <origin xyz="0 0 0" rpy="0 0 0"/>
+        <geometry>
+          <sphere radius="${caster_radius}"/>
+        </geometry>
+        <material name="caster_metallic"/>
+      </visual>
+      <!-- Caster mounting collar connecting to chassis underside -->
+      <visual>
+        <origin xyz="0 0 ${caster_radius * 0.7}" rpy="0 0 0"/>
+        <geometry>
+          <cylinder radius="${caster_radius * 0.75}" length="${caster_radius * 0.6}"/>
+        </geometry>
+        <material name="dark_grey"/>
+      </visual>
+      <collision>
+        <origin xyz="0 0 0" rpy="0 0 0"/>
+        <geometry>
+          <sphere radius="${caster_radius}"/>
+        </geometry>
+      </collision>
+      <!-- Solid sphere inertia tensor -->
+      <inertial>
+        <mass value="${caster_mass}"/>
+        <origin xyz="0 0 0" rpy="0 0 0"/>
+        <inertia
+          ixx="${(2.0 / 5.0) * caster_mass * caster_radius * caster_radius}"
+          ixy="0.0"
+          ixz="0.0"
+          iyy="${(2.0 / 5.0) * caster_mass * caster_radius * caster_radius}"
+          iyz="0.0"
+          izz="${(2.0 / 5.0) * caster_mass * caster_radius * caster_radius}"/>
+      </inertial>
+    </link>
+  </xacro:macro>
 </robot>
