Commit message: Added controls

File: src/ahser_description/urdf/ahser.urdf.xacro (robot description, xacro)
@@ -55,13 +55,13 @@
   <!-- Kinematic Base / Footprint Frames                                    -->
   <!-- ==================================================================== -->
-  <!-- Root Link: base_link located at ground plane projection of drive axle -->
-  <link name="base_link"/>
-  <!-- base_footprint on ground plane z=0 (REP 120 standard) -->
+  <!-- Root Link: base_footprint on ground plane z=0 (REP 120 standard) -->
+  <link name="base_footprint"/>
+  <!-- base_link located at ground plane projection of drive axle -->
   <joint name="base_footprint_joint" type="fixed">
-    <parent link="base_link"/>
-    <child link="base_footprint"/>
+    <parent link="base_footprint"/>
+    <child link="base_link"/>
     <origin xyz="0 0 0" rpy="0 0 0"/>
   </joint>
-  <link name="base_footprint"/>
+  <link name="base_link"/>
   <!-- ==================================================================== -->
   <!-- Main Chassis Link & Joint                                            -->
@@ -185,3 +185,37 @@
   <!-- ==================================================================== -->
   <xacro:sensors/>
+  <!-- ==================================================================== -->
+  <!-- Modern Gazebo (Jetty) Differential Drive & Joint State Plugins       -->
+  <!-- ==================================================================== -->
+  <gazebo>
+    <plugin
+      filename="gz-sim-diff-drive-system"
+      name="gz::sim::systems::DiffDrive">
+      <left_joint>left_wheel_joint</left_joint>
+      <right_joint>right_wheel_joint</right_joint>
+      <wheel_separation>${wheel_track}</wheel_separation>
+      <wheel_radius>${wheel_radius}</wheel_radius>
+      <max_linear_acceleration>1.5</max_linear_acceleration>
+      <min_linear_acceleration>-1.5</min_linear_acceleration>
+      <max_angular_acceleration>2.5</max_angular_acceleration>
+      <min_angular_acceleration>-2.5</min_angular_acceleration>
+      <max_linear_velocity>0.8</max_linear_velocity>
+      <min_linear_velocity>-0.8</min_linear_velocity>
+      <max_angular_velocity>1.5</max_angular_velocity>
+      <min_angular_velocity>-1.5</min_angular_velocity>
+      <topic>/cmd_vel</topic>
+      <odom_topic>/odom</odom_topic>
+      <tf_topic>/tf</tf_topic>
+      <frame_id>odom</frame_id>
+      <child_frame_id>base_footprint</child_frame_id>
+      <odom_publish_frequency>50</odom_publish_frequency>
+    </plugin>
+    <plugin
+      filename="gz-sim-joint-state-publisher-system"
+      name="gz::sim::systems::JointStatePublisher">
+      <topic>/joint_states</topic>
+      <joint_name>left_wheel_joint</joint_name>
+      <joint_name>right_wheel_joint</joint_name>
+    </plugin>
+  </gazebo>
 </robot>
